File: board/forkbomb19/forkbomb19.sch (EAGLE design)
At the start: 55 parts, among them SW1 SPST_TACT-KMR2, U1 ESP-WROOM-03, X3 POT_GND, X4 POT_3V3, X5 POT_SIG

Commit message: small board modifications
Parts:
- R1: value (none) -> 1k
Connections:
- net EN: now also U3G$1.#RST
Changed lines of the file:
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@@
 <?xml version="1.0" encoding="utf-8"?>
 <!DOCTYPE eagle SYSTEM "eagle.dtd">
-<eagle version="9.2.2">
+<eagle version="9.3.0">
 <drawing>
 <settings>
@@
 <part name="U2" library="forkbomb19" deviceset="MICROBUILDER_AMG8833" device=""/>
 <part name="HRDRST" library="SparkFun-Jumpers" library_urn="urn:adsk.eagle:library:528" deviceset="JUMPER-SMT_2_NO" device="_SILK_ROUND" package3d_urn="urn:adsk.eagle:package:39280/1" value=""/>
-<part name="R1" library="resistor" library_urn="urn:adsk.eagle:library:348" deviceset="R-US_" device="R0603" package3d_urn="urn:adsk.eagle:package:23555/2"/>
+<part name="R1" library="resistor" library_urn="urn:adsk.eagle:library:348" deviceset="R-US_" device="R0603" package3d_urn="urn:adsk.eagle:package:23555/2" value="1k"/>
 <part name="C1" library="resistor" library_urn="urn:adsk.eagle:library:348" deviceset="C-US" device="C0603" package3d_urn="urn:adsk.eagle:package:23616/2" value="100nF"/>
 <part name="GND1" library="supply1" library_urn="urn:adsk.eagle:library:371" deviceset="GND" device=""/>
@@
 <label x="180.34" y="30.48" size="1.778" layer="95" rot="R270"/>
 </segment>
+<segment>
+<pinref part="U3" gate="G$1" pin="#RST"/>
+<wire x1="139.7" y1="73.66" x2="147.32" y2="73.66" width="0.1524" layer="91"/>
+<label x="147.32" y="73.66" size="1.778" layer="95"/>
+<junction x="147.32" y="73.66"/>
+</segment>
 </net>
